File: astrodewar-mas-flex.kicad_pcb (KiCad board)
At the start: 2 copper layers, 287 x 67.3 mm, 2 parts, among them J1 Conn_02x25_Top_Bottom, U1 DB-50-LTA-V2

Commit message: Add files via upload
Routing:
- net H3C: track 524.7 -> 288.7 mm
- net SWC: track 512.9 -> 277.4 mm
- net OGC: track 509.8 -> 277.4 mm
- net H2C: track 510.6 -> 279.4 mm
- net V2C: track 503.2 -> 300.0 mm
- net VDD: track 481.3 -> 443.1 mm
- net VREF: track 478.6 -> 441.5 mm
- net VDRAIN: track 485.4 -> 455.7 mm
- net V3B: track 281.1 -> 282.1 mm
- net TGA: track 271.5 -> 270.9 mm
